File: AngularRGB.kicad_pcb (KiCad board)
At the start: 2 copper layers, 228.6 x 76.2 mm, 170 parts, among them J1 Conn_01x09_Male, SW1 SW_Push, SW1.25U1 MX_1.25U, SW1.25U2 MX_1.25U, SW1.25U3 MX_1.25U, SW1.25U4 MX_1.25U, SW1.25U5 MX_1.25U, SW1.25U6 MX_1.25U, SW1.75U1 MX_1.75U, SW1.75U2 MX_1.75U, SW10 MX_1U, SW11 MX_1U, SW12 MX_1U, SW13 MX_1U, SW14 MX_1U, SW15 MX_1U, SW16 MX_1U, SW17 MX_1U, SW18 MX_1U, SW19 MX_1U, SW2 MX_1U, SW2.25U1 MX_2.25U, SW2.75U1 MX_2.75U, SW20 MX_1U, SW21 MX_1U, SW22 MX_1U, SW23 MX_1U, SW24 MX_1U, SW25 MX_1U, SW26 MX_1U, SW27 MX_1U, SW28 MX_1U, SW29 MX_1U, SW3 MX_1U, SW30 MX_1U, SW31 MX_1U, SW32 MX_1U, SW33 MX_1U, SW4 MX_1U, SW5 MX_1U, SW6 MX_1U, SW7 MX_1U, SW8 MX_1U, SW9 MX_1U, U1 ATmega32U4-MU, U2 USB6B1, Y1 Crystal_GND24

Commit message: Added Case Design
Parts:
- removed J1: Conn_01x09_Male, Connector_PinSocket_2.54mm:PinSocket_1x09_P2.54mm_Vertical
- removed LED23, LED27, LED35: WS2812, MX_Switches:REVERSE_LED
- added ANT1: SWRA117D, RF_Antenna:Texas_SWRA117D_2.4GHz_Right, B.Cu at (319.8, 90.3)
- added C17: 1u, Capacitor_SMD:C_0603_1608Metric, B.Cu at (228.1, 79.4)
- added C18: 100n, Capacitor_SMD:C_0603_1608Metric, B.Cu at (301.6, 87.7)
- added C19: 100n, Capacitor_SMD:C_0603_1608Metric, B.Cu at (300.3, 96.4)
- added C20: 1u, Capacitor_SMD:C_0603_1608Metric, B.Cu at (238.1, 78.9)
- added C21: 1.5pF, Capacitor_SMD:C_0603_1608Metric, B.Cu at (317.1, 91.3)
- added C22: 1.0pF, Capacitor_SMD:C_0603_1608Metric, B.Cu at (312.7, 93.1)
- added C23: 2.2pF, Capacitor_SMD:C_0603_1608Metric, B.Cu at (311.2, 90.5)
- added C24: 12pF, Capacitor_SMD:C_0603_1608Metric, B.Cu at (310.2, 98.2)
- added C25: 100n, Capacitor_SMD:C_0603_1608Metric, B.Cu at (308.8, 88.3)
- added C26: 2.2nF, Capacitor_SMD:C_0603_1608Metric, B.Cu at (310.0, 95.6)
- added C27: 47n, Capacitor_SMD:C_0603_1608Metric, F.Cu at (307.2, 95.9)
- added C28: 12pF, Capacitor_SMD:C_0603_1608Metric, B.Cu at (304.4, 98.2)
- added C29: 1.0n, Capacitor_SMD:C_0603_1608Metric, F.Cu at (318.0, 97.8)
- added D43: D, Diode_SMD:D_SOD-123, B.Cu at (239.7, 90.2)
- added L1: 3.3nH, Inductor_SMD:L_0603_1608Metric, B.Cu at (314.5, 90.5)
- added L2: 4.7nH, Inductor_SMD:L_0603_1608Metric, B.Cu at (309.4, 92.0)
- added L3: 10nH, Inductor_SMD:L_0603_1608Metric, B.Cu at (310.7, 93.1)
- added Q1: BSS138, Package_TO_SOT_SMD:SOT-23, B.Cu at (229.0, 87.9)
- added R7: 5k1, Resistor_SMD:R_0603_1608Metric, B.Cu at (228.9, 84.6)
- added R8: 5k1, Resistor_SMD:R_0603_1608Metric, B.Cu at (229.1, 91.6)
- added R9: 5k1, Resistor_SMD:R_0603_1608Metric, B.Cu at (301.8, 98.9)
- added U3: 74LVC2G34, Package_TO_SOT_SMD:SOT-23-6, B.Cu at (234.9, 89.7)
- added U4: AMS1117-3.3, Package_TO_SOT_SMD:SOT-223-3_TabPin2, B.Cu at (233.4, 81.7)
- added U5: nRF51x22-QFxx, Package_DFN_QFN:QFN-48-1EP_6x6mm_P0.4mm_EP4.66x4.66mm, B.Cu at (304.6, 92.0)
- added Y2: Crystal_GND24, Crystal:Crystal_SMD_3225-4Pin_3.2x2.5mm, B.Cu at (307.3, 98.3)
- C4, C5: moved to F.Cu
- moved C3 38.1 mm to (116.6, 91.3)
- moved C6 35.4 mm to (110.6, 89.1), turned to 135 degrees
- moved C4 34.8 mm to (108.0, 93.6), turned to 0 degrees
- moved C5 34.8 mm to (105.0, 93.6), turned to 180 degrees
- moved Y1 32.4 mm to (113.2, 92.5), turned to 90 degrees
- moved C2 30.2 mm to (116.6, 93.6), turned to 0 degrees
- moved C7 28.7 mm to (100.7, 91.9)
- moved U1 26.8 mm to (106.6, 95.1), turned to 270 degrees
- moved C8 26.4 mm to (108.4, 102.1), turned to 0 degrees
- moved SW32 23.8 mm to (230.3, 101.7)
- moved C14 23.6 mm to (226.1, 60.7), turned to 270 degrees
- moved D39 19.4 mm to (243.4, 72.5), turned to 270 degrees
- moved H5 19.2 mm to (225.3, 92.2)
- moved SW1.25U5 19.0 mm to (251.7, 101.7)
- moved C12 14.9 mm to (244.6, 116.1), turned to 90 degrees
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Connections:
- LED31 pad 4: Net-(LED27-Pad2) -> Net-(LED19-Pad2)
- LED39 pad 4: Net-(LED35-Pad2) -> Net-(LED31-Pad2)
- SW1.25U5 pad 2: Net-(D36-Pad2) -> Net-(D40-Pad2)
- SW32 pad 2: Net-(D40-Pad2) -> Net-(D36-Pad2)
Routing:
- net VCC: track 1307.7 -> 0.00 mm, vias 54 -> 0
- net R0: track 275.6 -> 0.00 mm, vias 3 -> 0
- net R1: track 245.4 -> 0.00 mm, vias 3 -> 0
- net Net-(LED2-Pad4): track 238.3 -> 0.00 mm, vias 2 -> 0
- net Net-(LED4-Pad4): track 238.1 -> 0.00 mm, vias 6 -> 0
- net R2: track 228.4 -> 0.00 mm, vias 6 -> 0
- net Net-(LED3-Pad4): track 228.3 -> 0.00 mm, vias 2 -> 0
- net R3: track 222.0 -> 0.00 mm, vias 1 -> 0
- net C11: track 219.0 -> 0.00 mm, vias 2 -> 0
- net C10: track 185.8 -> 0.00 mm, vias 2 -> 0
- net C9: track 172.0 -> 0.00 mm, vias 2 -> 0
- net C8: track 142.1 -> 0.00 mm, vias 2 -> 0
- net C0: track 139.6 -> 0.00 mm, vias 5 -> 0
- net LED_INPUT: track 121.9 -> 0.00 mm, vias 8 -> 0
- net C7: track 118.8 -> 0.00 mm, vias 3 -> 0
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- removed copper zone on B.Cu, net GND
- removed copper zone on F.Cu, net GND
Other:
- copper layers 2 -> 4
- net class Default: clearance 0.153 -> 0.15
- rule trace_clearance: 0.153 -> 0.15
- board text removed: "CS"
- board text removed: "IRQ"
- board text removed: "MISO"
- board text removed: "MOSI"
- board text removed: "NC"
- board text removed: "RST"
- board text removed: "SCK"
- board text removed: "VCC"
