File: AngularRGB.sch (KiCad schematic (older format))
At the start: 170 parts, among them J1 Conn_01x09_Male, SW1 SW_Push, SW1.25U1 MX_1.25U, SW1.25U2 MX_1.25U, SW1.25U3 MX_1.25U, SW1.25U4 MX_1.25U, SW1.25U5 MX_1.25U, SW1.25U6 MX_1.25U, SW1.75U1 MX_1.75U, SW1.75U2 MX_1.75U, SW10 MX_1U, SW11 MX_1U, SW12 MX_1U, SW13 MX_1U, SW14 MX_1U, SW15 MX_1U, SW16 MX_1U, SW17 MX_1U, SW18 MX_1U, SW19 MX_1U, SW2 MX_1U, SW2.25U1 MX_2.25U, SW2.75U1 MX_2.75U, SW20 MX_1U, SW21 MX_1U, SW22 MX_1U, SW23 MX_1U, SW24 MX_1U, SW25 MX_1U, SW26 MX_1U, SW27 MX_1U, SW28 MX_1U, SW29 MX_1U, SW3 MX_1U, SW30 MX_1U, SW31 MX_1U, SW32 MX_1U, SW33 MX_1U, SW4 MX_1U, SW5 MX_1U, SW6 MX_1U, SW7 MX_1U, SW8 MX_1U, SW9 MX_1U, U1 ATmega32U4-MU, U2 USB6B1, Y1 Crystal_GND24

Commit message: Added Case Design
Parts:
- removed J1: Conn_01x09_Male, Connector_PinSocket_2.54mm:PinSocket_1x09_P2.54mm_Vertical, symbol Connector:Conn_01x09_Male
- removed LED23, LED27, LED35: WS2812, MX_Switches:REVERSE_LED, symbol MX_Switches:WS2812
- added ANT1: SWRA117D, RF_Antenna:Texas_SWRA117D_2.4GHz_Right, symbol MyAntennas:SWRA117D
- added C17, C20: 1u, Capacitor_SMD:C_0603_1608Metric, symbol Device:C
- added C18, C19, C25: 100n, Capacitor_SMD:C_0603_1608Metric, symbol Device:C
- added C21: 1.5pF, Capacitor_SMD:C_0603_1608Metric, symbol Device:C
- added C22: 1.0pF, Capacitor_SMD:C_0603_1608Metric, symbol Device:C
- added C23: 2.2pF, Capacitor_SMD:C_0603_1608Metric, symbol Device:C
- added C24, C28: 12pF, Capacitor_SMD:C_0603_1608Metric, symbol Device:C
- added C26: 2.2nF, Capacitor_SMD:C_0603_1608Metric, symbol Device:C
- added C27: 47n, Capacitor_SMD:C_0603_1608Metric, symbol Device:C
- added C29: 1.0n, Capacitor_SMD:C_0603_1608Metric, symbol Device:C
- added D43: D, Diode_SMD:D_SOD-123, symbol Device:D
- added L1: 3.3nH, Inductor_SMD:L_0603_1608Metric, symbol Device:L
- added L2: 4.7nH, Inductor_SMD:L_0603_1608Metric, symbol Device:L
- added L3: 10nH, Inductor_SMD:L_0603_1608Metric, symbol Device:L
- added Q1: BSS138, Package_TO_SOT_SMD:SOT-23, symbol Transistor_FET:BSS138
- added R7, R8, R9: 5k1, Resistor_SMD:R_0603_1608Metric, symbol Device:R
- added U3: 74LVC2G34, Package_TO_SOT_SMD:SOT-23-6, symbol MX_Switches:74LVC2G34
- added U4: AMS1117-3.3, Package_TO_SOT_SMD:SOT-223-3_TabPin2, symbol Regulator_Linear:AMS1117-3.3
- added U5: nRF51x22-QFxx, Package_DFN_QFN:QFN-48-1EP_6x6mm_P0.4mm_EP4.66x4.66mm, symbol MCU_Nordic:nRF51x22-QFxx
- added Y2: Crystal_GND24, Crystal:Crystal_SMD_3225-4Pin_3.2x2.5mm, symbol Device:Crystal_GND24
Connections:
- net CS: now also D43.1 (K)
- net GND: now also ANT1.2 (GND), C17.2, C18.2, C19.2, C20.2, C21.2, C22.2, C24.2, C25.2, C26.2, C27.2, C28.2, C29.2, U3.2 (GND), U4.1 (GND), U5.13 (VSS), U5.33 (VSS), U5.34 (VSS), U5.49 (EP), Y2.2, Y2.4
- net MISO: now also U5.41 (P0.22)
- net MOSI: now also U3.3 (2A)
- net RST: now also Q1.3 (D), R8.2
- net SCK: now also U3.1 (1A)
- net VCC: now also C17.1, R8.1, U4.3 (VI)
- net at D36.2 (A): now also SW32.2; no longer SW1.25U5.2
- net at D40.2 (A): now also SW1.25U5.2; no longer SW32.2
- net at LED19.2 (DO): now also LED31.4 (DI)
- net at LED39.4 (DI): now also LED31.2 (DO)
- new net: C25.1, U5.29 (DEC2)
- new net: C27.1, U5.39 (DEC1)
- new net: C22.1, C23.2, L1.2
- new net +3V3: C18.1, C19.1, C20.1, C29.1, Q1.1 (G), R7.1, R9.1, U3.5 (VCC), U4.2 (VO), U5.1 (VDD), U5.12 (VDD), U5.35 (AVDD), U5.36 (AVDD)
- new net ANT: ANT1.1 (SIG), C21.1, L1.1
- new net ANT1: C23.1, L2.1, U5.31 (ANT1)
- new net ANT2: L2.2, L3.1, U5.32 (ANT2)
- new net CONN: U5.27 (P0.19)
- new net CS_3V: D43.2 (A), R9.2, U5.43 (P0.24)
- new net DFU_3V: U5.11 (P0.7)
- new net FACTORYRST: U5.22 (P0.16)
- new net IRQ_3V: U5.44 (P0.25)
- new net MODE: U5.26 (P0.18)
- new net MOSI_3V: U3.4 (2Y), U5.42 (P0.23)
- new net SCK_3V: U3.6 (1Y), U5.40 (P0.21)
- new net SWDCLK: U5.24 (SWDCLK)
- new net SWDIO: Q1.2 (S), R7.2, U5.23 (SWDIO/~RST)
- new net VDD_PA: C26.1, L3.2, U5.30 (VDD_PA)
- new net XC1: C24.1, U5.37 (XC1), Y2.1
- new net XC2: C28.1, U5.38 (XC2), Y2.3
Other:
- moved on the sheet: C10, C11, C12, C13, C14, C15, C16, C9, LED1, LED10, LED11, LED12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
