File: Rev1.kicad_pcb (KiCad board)
At the start: 4 copper layers, 228.6 x 76.2 mm, 192 parts, among them Q1 BSS138, SW1 SW_Push, SW1.25U1 MX_1.25U, SW1.25U2 MX_1.25U, SW1.25U3 MX_1.25U, SW1.25U4 MX_1.25U, SW1.25U5 MX_1.25U, SW1.25U6 MX_1.25U, SW1.75U1 MX_1.75U, SW1.75U2 MX_1.75U, SW10 MX_1U, SW11 MX_1U, SW12 MX_1U, SW13 MX_1U, SW14 MX_1U, SW15 MX_1U, SW16 MX_1U, SW17 MX_1U, SW18 MX_1U, SW19 MX_1U, SW2 MX_1U, SW2.25U1 MX_2.25U, SW2.75U1 MX_2.75U, SW20 MX_1U, SW21 MX_1U, SW22 MX_1U, SW23 MX_1U, SW24 MX_1U, SW25 MX_1U, SW26 MX_1U, SW27 MX_1U, SW28 MX_1U, SW29 MX_1U, SW3 MX_1U, SW30 MX_1U, SW31 MX_1U, SW32 MX_1U, SW33 MX_1U, SW4 MX_1U, SW5 MX_1U, SW6 MX_1U, SW7 MX_1U, SW8 MX_1U, SW9 MX_1U, U1 ATmega32U4-MU, U2 USB6B1, U3 74LVC2G34, U4 AMS1117-3.3, U5 nRF51x22-QFxx, Y1 Crystal_GND24, Y2 Crystal_GND24

Commit message: Added Case Design
Parts:
- removed ANT1: SWRA117D, RF_Antenna:Texas_SWRA117D_2.4GHz_Right
- removed C17, C20: 1u, Capacitor_SMD:C_0603_1608Metric
- removed C18, C19, C25: 100n, Capacitor_SMD:C_0603_1608Metric
- removed C21: 1.5pF, Capacitor_SMD:C_0603_1608Metric
- removed C22: 1.0pF, Capacitor_SMD:C_0603_1608Metric
- removed C23: 2.2pF, Capacitor_SMD:C_0603_1608Metric
- removed C24, C28: 12pF, Capacitor_SMD:C_0603_1608Metric
- removed C26: 2.2nF, Capacitor_SMD:C_0603_1608Metric
- removed C27: 47n, Capacitor_SMD:C_0603_1608Metric
- removed C29: 1.0n, Capacitor_SMD:C_0603_1608Metric
- removed D43: D, Diode_SMD:D_SOD-123
- removed L1: 3.3nH, Inductor_SMD:L_0603_1608Metric
- removed L2: 4.7nH, Inductor_SMD:L_0603_1608Metric
- removed L3: 10nH, Inductor_SMD:L_0603_1608Metric
- removed Q1: BSS138, Package_TO_SOT_SMD:SOT-23
- removed R7, R8, R9: 5k1, Resistor_SMD:R_0603_1608Metric
- removed U3: 74LVC2G34, Package_TO_SOT_SMD:SOT-23-6
- removed U4: AMS1117-3.3, Package_TO_SOT_SMD:SOT-223-3_TabPin2
- removed U5: nRF51x22-QFxx, Package_DFN_QFN:QFN-48-1EP_6x6mm_P0.4mm_EP4.66x4.66mm
- removed Y2: Crystal_GND24, Crystal:Crystal_SMD_3225-4Pin_3.2x2.5mm
- added J1: Conn_01x09_Male, Connector_PinSocket_2.54mm:PinSocket_1x09_P2.54mm_Vertical, B.Cu at (37.3, 111.3)
- added LED23: WS2812, MX_Switches:REVERSE_LED, F.Cu at (144.4, 120.6)
- added LED27: WS2812, MX_Switches:REVERSE_LED, F.Cu at (159.5, 120.6)
- added LED35: WS2812, MX_Switches:REVERSE_LED, F.Cu at (191.4, 120.6)
- C4, C5: moved to B.Cu
- moved C3 38.1 mm to (99.8, 125.5)
- moved C6 35.4 mm to (115.6, 124.1), turned to 90 degrees
- moved C4 34.8 mm to (111.1, 128.3), turned to 180 degrees
- moved C5 34.8 mm to (108.1, 128.3), turned to 0 degrees
- moved Y1 32.4 mm to (99.9, 122.1), turned to 270 degrees
- moved C2 30.2 mm to (99.8, 118.7), turned to 180 degrees
- moved C7 28.7 mm to (114.0, 117.3)
- moved U1 26.8 mm to (108.0, 121.9), turned to 90 degrees
- moved C8 26.4 mm to (105.0, 128.3), turned to 180 degrees
- moved SW32 23.8 mm to (254.0, 101.6)
- moved C14 23.6 mm to (236.2, 82.0), turned to 90 degrees
- moved D39 19.4 mm to (249.3, 90.9), turned to 180 degrees
- moved H5 19.2 mm to (244.5, 92.1)
- moved SW1.25U5 19.0 mm to (232.7, 101.7)
- moved C12 14.9 mm to (244.2, 101.2), turned to 270 degrees
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Connections:
- LED31 pad 4: Net-(LED19-Pad2) -> Net-(LED27-Pad2)
- LED39 pad 4: Net-(LED31-Pad2) -> Net-(LED35-Pad2)
- SW1.25U5 pad 2: Net-(D40-Pad2) -> Net-(D36-Pad2)
- SW32 pad 2: Net-(D36-Pad2) -> Net-(D40-Pad2)
Routing:
- net VCC: track 0.00 -> 1307.7 mm, vias 0 -> 54
- net R0: track 0.00 -> 275.6 mm, vias 0 -> 3
- net R1: track 0.00 -> 245.4 mm, vias 0 -> 3
- net Net-(LED2-Pad4): track 0.00 -> 238.3 mm, vias 0 -> 2
- net Net-(LED4-Pad4): track 0.00 -> 238.1 mm, vias 0 -> 6
- net R2: track 0.00 -> 228.4 mm, vias 0 -> 6
- net Net-(LED3-Pad4): track 0.00 -> 228.3 mm, vias 0 -> 2
- net R3: track 0.00 -> 222.0 mm, vias 0 -> 1
- net C11: track 0.00 -> 219.0 mm, vias 0 -> 2
- net C10: track 0.00 -> 185.8 mm, vias 0 -> 2
- net C9: track 0.00 -> 172.0 mm, vias 0 -> 2
- net C8: track 0.00 -> 142.1 mm, vias 0 -> 2
- net C0: track 0.00 -> 139.6 mm, vias 0 -> 5
- net LED_INPUT: track 0.00 -> 121.9 mm, vias 0 -> 8
- net C7: track 0.00 -> 118.8 mm, vias 0 -> 3
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Other:
- copper layers 4 -> 2
- net class Default: clearance 0.15 -> 0.153
- rule trace_clearance: 0.15 -> 0.153
- board text added: "CS"
- board text added: "IRQ"
- board text added: "MISO"
- board text added: "MOSI"
- board text added: "NC"
- board text added: "RST"
- board text added: "SCK"
- board text added: "VCC"
